File: PCB Design/Box PCB/box''.brd (EAGLE design)
At the start: 50 x 65 mm, 12 parts

Commit message: schematic and gui changes
Parts:
- removed JP7: (no value), SparkFun:1X01
Connections:
- net S$10: no longer JP7.1
Routing:
- net S$10: track 59.1 -> 57.8 mm
- net S$8: track 21.0 -> 20.4 mm
Changed lines of the file:
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@@
 <element name="JP4" library="SparkFun" package="1X01" value="" x="38.989" y="27.6822" rot="MR0"/>
 <element name="E$1" library="audiojack" package="SMDAUDIO" value="" x="0" y="14.5"/>
-<element name="JP7" library="SparkFun" package="1X01" value="" x="19.489" y="12.1422" rot="MR0"/>
 <element name="E$2" library="discrete" package="R-5" value="" x="19.5" y="22" rot="R90"/>
 <element name="JP8" library="SparkFun" package="1X01" value="" x="30.489" y="62.6422" rot="MR0"/>
@@
 </signal>
 <signal name="S$10">
-<contactref element="JP7" pad="1"/>
-<contactref element="JP6" pad="12"/>
-<wire x1="41.91" y1="18.97" x2="42" y2="18.97" width="0.4064" layer="16"/>
-<wire x1="42" y1="18.97" x2="42" y2="11.5" width="0.4064" layer="16"/>
-<wire x1="42" y1="11.5" x2="19.489" y2="11.5" width="0.4064" layer="16"/>
-<wire x1="19.489" y1="11.5" x2="19.489" y2="12.1422" width="0.4064" layer="16"/>
 <contactref element="E$1" pad="P$1"/>
 <wire x1="1.7" y1="15.975" x2="1.7" y2="13.3" width="0.4064" layer="1"/>
@@
 <wire x1="19.489" y1="12.1422" x2="19.489" y2="19.449" width="0.4064" layer="1"/>
 <wire x1="19.489" y1="19.449" x2="19.5" y2="19.46" width="0.4064" layer="1"/>
+<contactref element="JP6" pad="12"/>
+<wire x1="41.91" y1="18.97" x2="41.91" y2="12.91" width="0.4064" layer="1"/>
+<wire x1="41.91" y1="12.91" x2="40.5" y2="11.5" width="0.4064" layer="1"/>
+<wire x1="40.5" y1="11.5" x2="19.8468" y2="11.5" width="0.4064" layer="1"/>
+<wire x1="19.8468" y1="11.5" x2="19.3468" y2="12" width="0.4064" layer="1"/>
 </signal>
 <signal name="S$7">
@@
 <contactref element="JP9" pad="1"/>
 <contactref element="JP6" pad="1"/>
-<wire x1="41.91" y1="46.91" x2="44.41" y2="46.91" width="0.4064" layer="1"/>
-<wire x1="44.41" y1="46.91" x2="45" y2="47.5" width="0.4064" layer="1"/>
-<wire x1="45" y1="47.5" x2="45" y2="56.6312" width="0.4064" layer="1"/>
-<wire x1="45" y1="56.6312" x2="38.989" y2="62.6422" width="0.4064" layer="1"/>
+<wire x1="41.91" y1="46.91" x2="43.41" y2="46.91" width="0.4064" layer="16"/>
+<wire x1="43.41" y1="46.91" x2="45" y2="48.5" width="0.4064" layer="16"/>
+<wire x1="45" y1="48.5" x2="45" y2="56.6312" width="0.4064" layer="16"/>
+<wire x1="45" y1="56.6312" x2="38.989" y2="62.6422" width="0.4064" layer="16"/>
 </signal>
 </signals>
